File: schematics/eight_by/eight_by.kicad_pcb (KiCad board)
At the start: 2 copper layers, 172.7 x 44.4 mm, 42 parts, among them J1 Conn_01x08, SW1 SW_Push_45deg, SW2 SW_Push_45deg, SW3 SW_Push_45deg, SW4 SW_Push_45deg, SW5 SW_Push_45deg, SW6 SW_Push_45deg, SW7 SW_Push_45deg, SW8 SW_Push_45deg, U1 74HC4051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

Commit message: pcb silkscren update
Parts:
- moved J1 4.58 mm to (27.6, 39.4)
- moved H2 3.59 mm to (29.2, 66.0)
- moved H4 3.59 mm to (194.3, 66.0)
- moved RV6 2.54 mm to (139.6, 42.9)
- moved RV7 2.54 mm to (160.0, 42.9)
- moved SW6 2.54 mm to (138.9, 51.4)
- moved SW7 2.54 mm to (159.2, 51.4)
- moved C5 2.54 mm to (87.6, 63.5)
- moved LED4 2.54 mm to (101.6, 63.5)
- moved RV3 2.54 mm to (78.7, 42.9)
- moved RV5 2.54 mm to (119.3, 42.9)
- moved SW3 2.54 mm to (77.9, 51.4)
- moved SW5 2.54 mm to (118.6, 51.4)
- moved C3 2.54 mm to (46.5, 63.5)
- moved H1 2.54 mm to (29.2, 29.2)
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Routing:
- net /NEOPIXEL: track 18.8 -> 14.4 mm
- net /SW: track 117.8 -> 113.8 mm
- net /POT: track 76.1 -> 72.6 mm
- net /S0: track 108.1 -> 109.7 mm
- net +3V3: track 287.1 -> 285.5 mm
- net /S1: track 107.1 -> 108.7 mm
Other:
- outline, holes or cut-outs redrawn
- board text added: "1"
- board text added: "2"
- board text added: "3"
- board text added: "4"
- board text added: "5"
- board text added: "6"
- board text added: "7"
- board text added: "8"
- board text added: "Gnd 3V3 Pot Sw S2 S1 S0 LEDs"
- board text added: "eight_by - @todbot"
- board text added: "eight_by - @todbot github.com/todbot/eight_by - 20 Jun 2024"

Commit message: eight_by_qtpy idea
Routing:
- net /POT7: track 105.5 -> 106.9 mm
- net /POT6: track 81.1 -> 82.2 mm
- net /POT2: track 67.9 -> 67.3 mm
- net /POT1: track 87.4 -> 88.0 mm
